File: Column Controller/Column Controller.kicad_pcb (KiCad board)
At the start: 4 copper layers, 105 x 72 mm, 187 parts, among them J1 B3B-XH-AM, J10 XT30, J11 XT30, J12 B5B-XH-AM, J13 XT30, J14 XT30, J15 XT30, J2 B3B-XH-AM, J3 B3B-XH-AM, J4 B4B-XH-AM, J5 XT30, J6 XT30, J7 B4B-XH-AM, J8 B4B-XH-AM, J9 XT30, Q1 BC817-25LT1G, Q2 BC817-25LT1G, Q3 DMN3404L, Q4 DMN3404L, Q5 DMN3404L, Q6 DMN3404L, Q7 NVMFS6H858NLT1G, Q8 NVMFS6H858NLT1G, Q9 DMN3404L, SW1 PTS526SK15SMTR2 LFS, SW2 PTS526SK15SMTR2 LFS, U10 DRV8874PWPR, U11 INA181A2, U2 ESP32-MINI-1, U4 DRV8874PWPR, U5 INA181A2, U6 LM5148RGYR, U8 LD1117S33TR_SOT223, U9 LD1117S50TR_SOT223

Commit message: Updated 3V3 rail on column board
Parts:
- moved TP14 10.8 mm to (143.0, 92.0)
- moved TP36 8.00 mm to (147.0, 88.0)
- moved TP19 1.00 mm to (134.0, 132.0)
- moved TP23 1.00 mm to (109.0, 131.0)
Routing:
- net 3V3: track 335.8 -> 297.1 mm, vias 15 -> 14
- net /Microcontroller/MOTOR_2.nSLEEP: track 68.7 -> 66.5 mm
- net /Ext Sensors/LOAD.DT: track 50.5 -> 49.4 mm, vias 1 -> 2
- net /Ext Sensors/LOAD.SCK: track 51.5 -> 50.4 mm, vias 1 -> 2
- net /Microcontroller/MOTOR_1.EN/IN1: track 84.8 -> 85.7 mm
- net GND: track 66.8 -> 66.0 mm, vias 485 -> 473
- net 24V: track 122.0 -> 122.7 mm, vias 54 -> 53
- net /Microcontroller/MOTOR_1.CURR: track 96.3 -> 96.9 mm
